File: hardware/bottom_power_motor/bottom_power_motor.kicad_sch (KiCad schematic)
At the start: 103 parts, among them J1 Power/Motor 6p, J2 J_STK_A, J3 J_STK_B, J4 Stern, Q1 P-FET 60V 60A, U1 L78L12, U2 TPS54360, U2_CB 100n, U2_CO 47u, U2_CZ 3n3, U2_D 60V 3A, U2_L 10u, U2_RC 10k, U2_RH 53k6, U2_RL 10k2, U2_RT_R 100k, U3 TLV62569, U4 TPS54360, U4_CB 100n, U4_CO 22u, U4_CZ 3n3, U4_D 60V 3A, U4_L 33u, U4_RC 10k, U4_RH 68k1, U4_RL 10k0, U4_RT_R 100k

Commit message: feat: Mid- und Top-Schaltplan, Stack-Pinout v0.3 als gemeinsame Quelle
Mid (26 Bauteile, 52 Netze) und Top (24 Bauteile, 51 Netze), beide wie das
Bottom-Board erzeugt und per kicad-cli-Netzliste rueckverglichen - BESTANDEN,
offene Pins nur auf expliziter Freigabeliste (Strapping, PSRAM-Pins 35-37,
SBU, Expander-INT).

Mid: ESP32-S3-WROOM-1 mit vollstaendiger GPIO-Zuordnung (im Kopf des
Generators dokumentiert), MAX3485 mit Fail-Safe-Bias und DNP-Terminierung,
steckbarer RS485-Anschluss, PCF8574 auf 0x20 mit Portbelegung == YAML,
Piezo-Treiber an 5V, EN-RC plus Reset- und Boot-Taster. Der KiCad-THVD1451D
ist die Vollduplex-Variante ohne DE/RE, deshalb MAX3485.

Top: USB-C (UFP, 5k1 an CC1/CC2 einzeln, USBLC6 an der Buchse), acht
Sicheltaster paarweise parallel, SHT4x, ST77916-Anschluss (Footprint
PLATZHALTER bis das reale Modul vermessen ist), Stern-Ausgang mit
High-Side-P-FET an STAR_EN, Radar-Steckplatz.

Stack-Pinout v0.3 in tools/stack_pinout.py - die einzige Quelle, von allen
drei Generatoren importiert, docs/03 daraus erzeugt. Zwei Korrekturen:
- USB D+/D- laufen jetzt DOCH durch den Stack (J_STK_A 34/36). Die alte
  Regel galt fuer den USB-UART-Baustein, den es seit dem Wechsel auf den
  nativen S3-USB nicht mehr gibt.
- Der Sternstecker J4 auf dem Bottom-Board widersprach der Frontplatte
  (Kabelausgang vorn) - entfernt, Stecker und Schalt-FET sitzen auf TOP,
  STAR_EN kommt vom Expander ueber den Stack.

YAML auf INA/INB umgestellt (vier ledc-Ausgaenge, Umpolung ueber die
Zweigwahl), esphome config valide; YAML-Pins maschinell gegen den
Mid-Schaltplan geprueft - konsistent.

Co-Authored-By: Claude Opus 5 <noreply@anthropic.com>
Claude-Session: https://claude.ai/code/session_017FTFDJW9R41k2WFeDRNE3w
Parts:
- removed J4: Stern, Connector_JST:JST_PH_B2B-PH-K_1x02_P2.00mm_Vertical, symbol Connector_Generic:Conn_01x02
Connections:
- net RS485_RE is gone; now on net RS485_DIR: J3.16 (Pin_16)
- net RS485_DE renamed RS485_DIR
- net RSV_A1 renamed STAR_EN
- net RSV_A3 renamed USB_DP
- net RSV_A5 renamed USB_DN
Other:
- moved on the sheet: C10, C_M1A_B, C_M1B_B, C_M1_CS, C_M1_F, C_M2A_B, C_M2B_B, C_M2_CS, C_M2_F, D_M1A_B, D_M1B_B, D_M2A_B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

Commit message: feat: Layouts aller drei Boards - platziert, vernetzt, DRC-sauber
Neuer Generator tools/gen_layouts.py erzeugt die drei .kicad_pcb komplett:
Outline, Bohrbild, Frontmarkierung, Antennen-Sperrflaeche, alle Footprints
mit Netzen aus den Schaltplan-Generatoren, PGND-Zonen beidseitig. Mechanisch
gebundene Teile exakt platziert (Stackverbinder deckungsgleich, Taster auf
den Sichel-Stoesselpositionen, USB-C am Rand, ESP32-Antenne an der
Frontkante, FET-Raster berechnet); Rest kollisionsfrei per Spiralsuche mit
Netznachbar-Heuristik. DRC (pcbnew.WriteDRCReport - kicad-cli kann das erst
ab KiCad 8): KEINE Platzierungsfehler auf allen drei Boards. Offen bleibt
das ROUTING - die Boards sind route-fertig, Leiterbahnen sind Handarbeit.

Die Kollisionspruefung fand einen echten Mechanikfehler: Bohrbild v2.
Die Bohrungen 120/240 Grad lagen ~2 mm neben den Sicheltasten-Stoesseln
(117/243) - Schraubenkopf trifft Taster. Auf r21,5 blockieren Stack-
verbinder, ESP32-Antenne und Leistungsstecker alle uebrigen Winkel; frei
sind exakt 0/180. Jetzt zwei Schrauben, Verdrehsicherung ueber die beiden
Stackverbinder. docs/04 und gen_boards nachgezogen.

Weitere Ausbeute der Iterationen (jede von DRC oder Kollisionspruefung
erzwungen): Stackverbinder auf x=+/-14,2 (Diagonaltaster!), Taster auf
Alps-SKRK-Footprint (EVQP2-Pads ragten 0,1 mm an den Rand), Rotations-
automatik fuer die Taster nach minimalem Pad-Radius, Sicherung auf
SMD-NANO2, Bulk-Elkos niedrigbauend auf die Rueckseite, Treiber gestaffelt
unter den FETs, HSOP ohne Thermal-Vias (0,2-mm-Bohrungen), Flip-Bug der
Autoplatzierung (Teile blieben nach B-Versuch gespiegelt), Segfault-
Workarounds fuer ZONE_FILLER und BOX2-Merge in der headless pcbnew-API.

Schaltplan-Nebenkorrekturen: L78L12-Pinbelegung war verdreht (1=OUT!),
Q1-Verpolschutz auf PowerPAK mit eigener Pad-Zuordnung, SHT4x-Footprint
lag in Sensor_Humidity statt Package_DFN_QFN.

USB-C-Randverletzungen (10) sind als Steckerueberhang beabsichtigt und
werden getrennt ausgewie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
Parts:
- C3, C4: value 470u/35V -> 220u/35V Polymer; footprint Capacitor_SMD:CP_Elec_10x10.5 -> Capacitor_SMD:CP_Elec_8x6.5
- F1: footprint Fuse:Fuse_Bourns_MF-RG300 -> Fuse:Fuse_Littelfuse-NANO2-451_453; MPN messabhaengig, siehe docs/11 -> SMD NANO2, messabhaengig - siehe docs/11
- J1: footprint Connector_Molex:Molex_Micro-Fit_3.0_43045-0600_2x03_P3.00mm_Vertical -> Connector_Molex:Molex_Micro-Fit_3.0_43045-0612_2x03_P3.00mm_Vertical
- L1: footprint Inductor_SMD:L_Bourns-SRP5030T -> Inductor_SMD:L_Bourns_SRP5030T
- Q1: value P-FET 60V 60A -> P-FET 40V 30A; footprint Package_TO_SOT_SMD:TO-263-2 -> Package_SO:PowerPAK_SO-8_Single; MPN z.B. IRF4905S - bestaetigen -> z.B. SiR429DP; Pad-Zuordnung siehe PAD_MAP in gen_layouts
- Q_M1A_H, Q_M1A_L, Q_M1B_H, Q_M1B_L, Q_M2A_H, Q_M2A_L, Q_M2B_H, Q_M2B_L: footprint Package_SO:SOIC-8_3.9x4.9mm_P1.27mm -> Package_SO:PowerPAK_SO-8_Single; MPN PowerPAK SO-8, Rds<5mOhm - Footprint bestaetigen -> Rds<5mOhm, z.B. SiR622DP - bestaetigen
- U2, U4: footprint Package_SO:HSOP-8-1EP_3.9x4.9mm_P1.27mm_EP2.4x3.2mm -> Package_SO:HSOP-8-1EP_3.9x4.9mm_P1.27mm_EP2.41x3.1mm
- U2_L, U4_L: footprint Inductor_SMD:L_Bourns-SRP7028A -> Inductor_SMD:L_Bourns_SRP7028A_7.3x6.6mm
Connections:
- net 12V_GATE: now also U1.1 (OUT); no longer U1.3 (IN)
- net 12V_RAW: now also U1.3 (IN); no longer U1.1 (OUT)
