File: hardware/bottom_power_motor/bottom_power_motor.kicad_sch (KiCad schematic)
At the start: 102 parts, among them J1 Power/Motor 6p, J2 J_STK_A, J3 J_STK_B, Q1 P-FET 40V 30A, U1 L78L12, U2 TPS54360, U2_CB 100n, U2_CO 47u, U2_CZ 3n3, U2_D 60V 3A, U2_L 10u, U2_RC 10k, U2_RH 53k6, U2_RL 10k2, U2_RT_R 100k, U3 TLV62569, U4 TPS54360, U4_CB 100n, U4_CO 22u, U4_CZ 3n3, U4_D 60V 3A, U4_L 33u, U4_RC 10k, U4_RH 68k1, U4_RL 10k0, U4_RT_R 100k

Commit message: docs/16: Anleitung fuer die letzten Handgriffe in KiCad
Was der Autorouter uebrig laesst, ist wenig und immer dasselbe Muster: Pads,
die zwischen anderen Bauteilen eingeklemmt sind. Die Anleitung nennt die
Tastenkuerzel (X fuer Bahn, V fuer Lagenwechsel mit Via, B fuer Zonen
fuellen), den aktuellen Stand je Board als Anhaltspunkt und die
Reihenfolge danach - Zonen fuellen VOR der DRC, sonst sucht man Fehler, die
keine sind.

Dazu zwei Warnungen: keine Bauteile verschieben, die Positionen kommen aus
gen_layouts.py und gehen beim naechsten Neuerzeugen verloren. Und die Regeln
nicht lockern - wenn die DRC meckert, ist die Bahn falsch.

Co-Authored-By: Claude Opus 5 (1M context) <noreply@anthropic.com>
Parts:
- removed C5, C6: 1u, Capacitor_SMD:C_0603_1608Metric, symbol Device:C
- removed C_M1A_B, C_M1B_B, C_M2A_B, C_M2B_B: 100n, Capacitor_SMD:C_0603_1608Metric, symbol Device:C
- removed D3: 27V, Diode_SMD:D_SOD-123, symbol Device:D_Zener
- removed D_M1A_B, D_M1B_B, D_M2A_B, D_M2B_B: 100V 1A, Diode_SMD:D_SOD-123, symbol Device:D_Schottky
- removed Q_M1A_H, Q_M1A_L, Q_M1B_H, Q_M1B_L, Q_M2A_H, Q_M2A_L, Q_M2B_H, Q_M2B_L: N-FET 40V 60A, Package_SO:PowerPAK_SO-8_Single, symbol SwitchStack:Q_NMOS_GDS
- removed R2: 100R, Resistor_SMD:R_0603_1608Metric, symbol Device:R
- removed R_M1A_HO, R_M1A_LO, R_M1B_HO, R_M1B_LO, R_M2A_HO, R_M2A_LO, R_M2B_HO, R_M2B_LO: 10R, Resistor_SMD:R_0603_1608Metric, symbol Device:R
- removed U1: L78L12, Package_TO_SOT_SMD:SOT-89-3, symbol Regulator_Linear:L78L12_SOT89
- removed UM1A_DRV, UM1B_DRV, UM2A_DRV, UM2B_DRV: IR2104, Package_SO:SOIC-8_3.9x4.9mm_P1.27mm, symbol Driver_FET:IR2104
- added C_M1_BR, C_M2_BR: 100u 50V, Capacitor_SMD:C_1210_3225Metric, symbol Device:C
- added R_M1_IL, R_M2_IL: 33k0, Resistor_SMD:R_0603_1608Metric, symbol Device:R
- added UM1_BR, UM2_BR: DRV8871, Package_SO:HSOP-8-1EP_3.9x4.9mm_P1.27mm_EP2.41x3.1mm_ThermalVias, symbol Driver_Motor:DRV8871DDA
- added UM1_GA, UM1_GB, UM2_GA, UM2_GB: 74AHC1G08, Package_TO_SOT_SMD:SOT-353_SC-70-5, symbol 74xGxx:74AHC1G08
- J1: value Power/Motor 6p -> Feld 16p; footprint Connector_Molex:Molex_Micro-Fit_3.0_43045-0612_2x03_P3.00mm_Vertical -> Connector_Molex:Molex_Micro-Fit_3.0_43045-1612_2x08_P3.00mm_Vertical; symbol Connector_Generic:Conn_02x03_Odd_Even -> Connector_Generic:Conn_02x08_Odd_Even; MPN Micro-Fit 3.0 2x3 - Strombelastbarkeit pruefen -> Molex 43045-1612, 2x8, stehend - EIN Stecker fuer alles, SE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
Connections:
- net 24V_PROT: now also C_M1_BR.1, C_M2_BR.1, UM1_BR.5 (VM), UM2_BR.5 (VM)
- net 3V3_SYS: now also UM1_GA.5 (VCC), UM1_GB.5 (VCC), UM2_GA.5 (VCC), UM2_GB.5 (VCC)
- net M1_B: now also UM1_BR.8 (OUT2)
- net M1_INA: now also UM1_GA.1
- net M1_INB: now also UM1_GB.1
- net M1_SD: now also UM1_GA.2, UM1_GB.2
- net M1_SWA: now also UM1_BR.6 (OUT1)
- net M2_B: now also UM2_BR.8 (OUT2)
- net M2_INA: now also UM2_GA.1
- net M2_INB: now also UM2_GB.1
- net M2_SD: now also UM2_GA.2, UM2_GB.2
- net M2_SWA: now also UM2_BR.6 (OUT1)
- net PGND: now also J1.16 (Pin_16), J1.7 (Pin_7), C_M1_BR.2, C_M2_BR.2, R_M1_IL.2, R_M2_IL.2, UM1_BR.1 (GND), UM1_BR.7 (GND), UM1_BR.9 (GND), UM1_GA.3 (GND), UM1_GB.3 (GND), UM2_BR.1 (GND), UM2_BR.7 (GND), UM2_BR.9 (GND), UM2_GA.3 (GND), UM2_GB.3 (GND); no longer J2.25 (Pin_25), J2.38 (Pin_38), J2.39 (Pin_39)
- net RSV_A2 renamed REED2_IN
- net REED2_IN: now also J1.12 (Pin_12)
- net RSV_A3 renamed RS485_A
- net RS485_A: now also J1.8 (Pin_8)
- net RSV_A4 renamed RS485_B
- net RS485_B: now also J1.9 (Pin_9)
- net RSV_A5 renamed REED1_IN
- net REED1_IN: now also J1.10 (Pin_10)
- net RSV_A6 renamed SAB1_IN
- net SAB1_IN: now also J1.11 (Pin_11)
- new net HOOD_A: J1.14 (Pin_14), J2.38 (Pin_38)
- new net HOOD_B: J1.15 (Pin_15), J2.39 (Pin_39)
- new net M1_GA: UM1_BR.3 (IN1), UM1_GA.4
- new net M1_GB: UM1_BR.2 (IN2), UM1_GB.4
- new net M1_ILIM: R_M1_IL.1, UM1_BR.4 (ILIM)
- new net M2_GA: UM2_BR.3 (IN1), UM2_GA.4
- new net M2_GB: UM2_BR.2 (IN2), UM2_GB.4
- new net M2_ILIM: R_M2_IL.1, UM2_BR.4 (ILIM)
- new net SAB2_IN: J1.13 (Pin_13), J2.25 (Pin_25)
Other:
- moved on the sheet: C10, C7, C8, C9, C_M1_CS, C_M1_F, C_M2_CS, C_M2_F, D4, D5, F2, J2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
